File: hardware/control_card.kicad_pcb (KiCad board)
At the start: 6 copper layers, 32.5 x 33.8 mm, 144 parts, among them J1 Power board, J2 JTAG, U1 A3CZ065BB18AE7S, U10 SN74LV4051APWR, U11 OPA365AIDBVR, U12 ADS7056IRUGR, U13 SN74LV4051APWR, U14 OPA365AIDBVR, U15 ADS7056IRUGR, U16 TLV75518PDBVR, U2 AP61302Z6-7, U3 AP61102Z6-7, U4 AP61102Z6-7, U5 TLV75512PDBVR, U6 TLV75533PDBVR, U7 MT25QU256ABA8E12-1SIT, U8 SN74AVC4T774RSVR, U9 W958D8NBYA5I, X1 100MHz

Commit message: 0.75 V buck: bottom-layer +0V75, GND and SW_0V75 zones
- B.Cu zones at the core buck: +0V75 over C3.1, C2.1 and L1.2; GND over
  C3.2/C2.2 and their vias; SW_0V75 from L1.1 to U2.4, kept narrow. Priority 5,
  0.2 mm clearance, solid pad connection, as at the 1.8 V buck.
- Includes hand edits made in KiCad since ffc3a6f.

DRC: 0 errors, 0 unconnected, 0 parity issues; 30 silkscreen warnings.

Co-Authored-By: Claude Opus 5.5 <noreply@anthropic.com>
Parts:
- moved C27 11.1 mm to (91.6, 113.0)
- moved C26 10.3 mm to (91.3, 115.0), turned to 0 degrees
- moved C28 9.18 mm to (93.5, 112.6), turned to 0 degrees
- moved C36 7.57 mm to (89.7, 114.9), turned to 180 degrees
- moved C35 5.03 mm to (90.1, 117.6), turned to -90 degrees
- moved C3 3.49 mm to (100.4, 110.5)
- moved R2 2.14 mm to (105.9, 116.4), turned to -90 degrees
- moved C19 1.72 mm to (89.4, 119.0), turned to 180 degrees
- moved R1 0.89 mm to (104.7, 114.7), turned to 90 degrees
- moved C39 0.07 mm to (89.4, 117.6)
Routing:
- net +0V75: track 20.8 -> 14.8 mm, vias 38 -> 37
- net /Power/FB_0V75: track 5.45 -> 3.20 mm
- net VCC_SENSE_N: track 15.4 -> 17.5 mm
- net GND: track 72.3 -> 70.7 mm, vias 179 -> 177
- net +1V8: track 15.8 -> 15.3 mm, vias 33 -> 31
- added copper zone on B.Cu, net +0V75
- added copper zone on B.Cu, net /Power/SW_0V75
