File: hardware/control_card.kicad_pcb (KiCad board)
At the start: 6 copper layers, 32.5 x 33.8 mm, 144 parts, among them J1 Power board, J2 JTAG, U1 A3CZ065BB18AE7S, U10 SN74LV4051APWR, U11 OPA365AIDBVR, U12 ADS7056IRUGR, U13 SN74LV4051APWR, U14 OPA365AIDBVR, U15 ADS7056IRUGR, U16 TLV75518PDBVR, U2 AP61302Z6-7, U3 AP61102Z6-7, U4 AP61102Z6-7, U5 TLV75512PDBVR, U6 TLV75533PDBVR, U7 MT25QU256ABA8E12-1SIT, U8 SN74AVC4T774RSVR, U9 W958D8NBYA5I, X1 100MHz

Commit message: start doing route cleanup
Routing:
- net /Configuration/AS_DATA1: track 11.2 -> 19.5 mm
- net /Configuration/AS_DATA0: track 11.3 -> 19.3 mm
- net /Configuration/AS_CLK: track 18.6 -> 22.9 mm
- net /Configuration/AS_NCS_MSEL0: track 15.9 -> 20.0 mm
- net /Configuration/TMS: track 5.63 -> 7.97 mm
- net /Configuration/TDO: track 4.66 -> 6.48 mm
- net /Configuration/TDI: track 6.50 -> 8.22 mm
- net +5V: track 82.8 -> 81.1 mm
- net HR_RWDS: track 7.35 -> 8.85 mm
- net /Configuration/TCK_1V8: track 10.9 -> 12.3 mm
- net HR_DQ3: track 7.57 -> 8.49 mm
- net HR_CS_N: track 7.93 -> 8.78 mm
- net HR_CK: track 6.32 -> 7.14 mm
- net /Configuration/AS_DATA3: track 23.9 -> 23.1 mm
- net GND: track 70.7 -> 70.0 mm, vias 177 -> 178
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