File: hardware/control_card.kicad_pcb (KiCad board)
At the start: 6 copper layers, 32.5 x 33.8 mm, 164 parts, among them J1 Power board, J2 JTAG, U1 A3CZ065BB18AE7S, U10 SN74LV4051APWR, U11 OPA365AIDBVR, U12 ADS7056IRUGR, U13 SN74LV4051APWR, U14 OPA365AIDBVR, U15 ADS7056IRUGR, U17 AP61102Z6-7, U18 AP61102Z6-7, U2 AP61302Z6-7, U3 AP61102Z6-7, U4 AP61102Z6-7, U6 TLV75533PDBVR, U7 MT25QU256ABA8E12-1SIT, U8 SN74AVC4T774RSVR, U9 W958D8NBYA5I, X1 100MHz

Commit message: Switcher pours, GND to U2/U17/U18 pins, R46 0201 part
B.Cu zones for the SW, output, GND and +5V nodes of all four AP61x02 cells,
with distinct priorities (equal-priority overlaps hang the KiCad 10 filler).
Ground pours extended to the switcher GND pins. Removed a dangling GND stub,
a PG_0V75 via in U2's pad and a dangling +1V2 via; reference designators
hidden again. R46 sits on an 0201 footprint: part changed to 0201WMF1003TEE
(C270364). DRC: 0 errors, 0 unconnected, 0 parity issues.

Co-Authored-By: Claude Opus 5.5 <noreply@anthropic.com>
Routing:
- net /Power/PG_1V8: track 52.7 -> 48.2 mm
- net +1V8_HR: track 10.9 -> 15.0 mm, vias 7 -> 9
- net +0V75: track 17.6 -> 20.3 mm, vias 32 -> 35
- net /Configuration/TMS: track 7.97 -> 6.84 mm
- net +3V3A: track 43.8 -> 42.9 mm
- net ADB6: track 11.3 -> 10.8 mm
- net /ADC/MUXB_OUT: track 2.70 -> 2.16 mm
- net /ADC/MUXA_OUT: track 4.33 -> 3.80 mm
- net ADB5: track 11.1 -> 10.5 mm
- net ADB3: track 4.88 -> 4.37 mm
- net /Power/PG_0V75: vias 3 -> 2
- net +1V2: vias 12 -> 11
- added copper zone on B.Cu, net +0V75
- added copper zone on B.Cu, net +1V2
- added copper zone on B.Cu, net +1V8_HR
- added copper zone on B.Cu, net +3V3
- added copper zone on B.Cu, net +5V
- added copper zone on B.Cu, net /Power/SW_0V75
- added copper zone on B.Cu, net /Power/SW_1V2
- added copper zone on B.Cu, net /Power/SW_1V8HR
- added copper zone on B.Cu, net /Power/SW_3V3
- added copper zone on B.Cu, net GND
