File: hardware/sheets/fpga_power.kicad_sch (KiCad schematic)
At the start: 45 parts, among them U1 A3CZ065BB18AE7S

Commit message: Replace two capacitors oversold at JLC
- C21-C23, C30, C31, C45 (4.7uF 0201 6.3V X5R): GRM035R60J475ME15D
  (C335103, -6875 orderable, min 127) -> Taiyo Yuden JDK063BBJ475MV-AT
  (C2880368, 109712 orderable, min 1).
- C65, C67, C69, C71 (47uF 0603 6.3V X5R): CGA0603X5R476M6R3JT
  (C6119831, -979 orderable, min 97) -> Murata GRM188R60J476ME15D
  (C140782, 124695 orderable, min 1).

Schematic and board updated together. All BOM parts now orderable for 10
boards with min purchase 1; tightest ADS7056 (29 orderable, 2 per board).
DRC: 0 errors, 0 unconnected, 0 parity issues.

Co-Authored-By: Claude Opus 5.5 <noreply@anthropic.com>
Parts:
- C21, C22, C23, C30, C31, C45: LCSC C335103 -> C2880368; MPN GRM035R60J475ME15D -> JDK063BBJ475MV-AT
- C65, C67, C69, C71: LCSC C6119831 -> C140782; MPN CGA0603X5R476M6R3JT -> GRM188R60J476ME15D
Changed lines of the file:
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@@
 			)
 		)
-		(property "LCSC" "C6119831"
+		(property "LCSC" "C140782"
 			(at 35.56 276.86 0)
 			(hide yes)
@@
 			)
 		)
-		(property "MPN" "CGA0603X5R476M6R3JT"
+		(property "MPN" "GRM188R60J476ME15D"
 			(at 35.56 276.86 0)
 			(hide yes)
@@
 			)
 		)
-		(property "LCSC" "C335103"
+		(property "LCSC" "C2880368"
 			(at 78.74 200.66 0)
 			(hide yes)
@@
 			)
 		)
-		(property "MPN" "GRM035R60J475ME15D"
+		(property "MPN" "JDK063BBJ475MV-AT"
 			(at 78.74 200.66 0)
 			(hide yes)
@@
 			)
 		)
-		(property "LCSC" "C335103"
+		(property "LCSC" "C2880368"
 			(at 104.14 200.66 0)
 			(hide yes)
@@
 			)
 		)
-		(property "MPN" "GRM035R60J475ME15D"
+		(property "MPN" "JDK063BBJ475MV-AT"
 			(at 104.14 200.66 0)
 			(hide yes)
@@
 			)
 		)
-		(property "LCSC" "C335103"
+		(property "LCSC" "C2880368"
 			(at 40.64 251.46 0)
 			(hide yes)
@@
 			)
 		)
-		(property "MPN" "GRM035R60J475ME15D"
+		(property "MPN" "JDK063BBJ475MV-AT"
 			(at 40.64 251.46 0)
 			(hide yes)
@@
 			)
 		)
-		(property "LCSC" "C6119831"
+		(property "LCSC" "C140782"
 			(at 134.62 276.86 0)
 			(hide yes)
@@
 			)
 		)
-		(property "MPN" "CGA0603X5R476M6R3JT"
+		(property "MPN" "GRM188R60J476ME15D"
 			(at 134.62 276.86 0)
 			(hide yes)
@@
 			)
 		)
-		(property "LCSC" "C6119831"
+		(property "LCSC" "C140782"
 			(at 101.6 276.86 0)
 			(hide yes)
@@
 			)
 		)
-		(property "MPN" "CGA0603X5R476M6R3JT"
+		(property "MPN" "GRM188R60J476ME15D"
 			(at 101.6 276.86 0)
 			(hide yes)
@@
 			)
 		)
-		(property "LCSC" "C335103"
+		(property "LCSC" "C2880368"
 			(at 53.34 226.06 0)
 			(hide yes)
@@
 			)
 		)
-		(property "MPN" "GRM035R60J475ME15D"
+		(property "MPN" "JDK063BBJ475MV-AT"
 			(at 53.34 226.06 0)
 			(hide yes)
@@
 			)
 		)
-		(property "LCSC" "C335103"
+		(property "LCSC" "C2880368"
 			(at 40.64 226.06 0)
 			(hide yes)
@@
 			)
 		)
-		(property "MPN" "GRM035R60J475ME15D"
+		(property "MPN" "JDK063BBJ475MV-AT"
 			(at 40.64 226.06 0)
 			(hide yes)
@@
 			)
 		)
-		(property "LCSC" "C6119831"
+		(property "LCSC" "C140782"
 			(at 68.58 276.86 0)
 			(hide yes)
@@
 			)
 		)
-		(property "MPN" "CGA0603X5R476M6R3JT"
+		(property "MPN" "GRM188R60J476ME15D"
 			(at 68.58 276.86 0)
 			(hide yes)
@@
 			)
 		)
-		(property "LCSC" "C335103"
+		(property "LCSC" "C2880368"
 			(at 91.44 200.66 0)
 			(hide yes)
@@
 			)
 		)
-		(property "MPN" "GRM035R60J475ME15D"
+		(property "MPN" "JDK063BBJ475MV-AT"
 			(at 91.44 200.66 0)
 			(hide yes)
