File: hardware/sheets/adc.kicad_sch (KiCad schematic)
At the start: 24 parts, among them U10 SN74LV4051APWR, U11 OPA365AIDBVR, U12 ADS7056IRUGR, U13 SN74LV4051APWR, U14 OPA365AIDBVR, U15 ADS7056IRUGR

Commit message: 33 ohm series resistors on 0201 pads: order the 0201 part
R27-R29 and R31-R33 sit on 0201 footprints but still carried the 0402
0402WGF330JTCE (C25105), so JLC would have placed 0402 parts on 0201 pads.
LCSC and MPN set to RC-01W33R0FT (C320843, 0201, 33 ohm 1 %) in the schematic
and on the board. Every other BOM line's footprint matches its JLC package.

DRC: 0 errors, 0 unconnected, 0 parity issues.

Co-Authored-By: Claude Opus 5.5 <noreply@anthropic.com>
Parts:
- R27, R28, R29, R31, R32, R33: LCSC C25105 -> C320843; MPN 0402WGF330JTCE -> RC-01W33R0FT
Changed lines of the file:
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@@
 			)
 		)
-		(property "LCSC" "C25105"
+		(property "LCSC" "C320843"
 			(at 104.14 177.8 0)
 			(hide yes)
@@
 			)
 		)
-		(property "MPN" "0402WGF330JTCE"
+		(property "MPN" "RC-01W33R0FT"
 			(at 104.14 177.8 0)
 			(hide yes)
@@
 			)
 		)
-		(property "LCSC" "C25105"
+		(property "LCSC" "C320843"
 			(at 129.54 88.9 0)
 			(hide yes)
@@
 			)
 		)
-		(property "MPN" "0402WGF330JTCE"
+		(property "MPN" "RC-01W33R0FT"
 			(at 129.54 88.9 0)
 			(hide yes)
@@
 			)
 		)
-		(property "LCSC" "C25105"
+		(property "LCSC" "C320843"
 			(at 104.14 88.9 0)
 			(hide yes)
@@
 			)
 		)
-		(property "MPN" "0402WGF330JTCE"
+		(property "MPN" "RC-01W33R0FT"
 			(at 104.14 88.9 0)
 			(hide yes)
@@
 			)
 		)
-		(property "LCSC" "C25105"
+		(property "LCSC" "C320843"
 			(at 119.38 177.8 0)
 			(hide yes)
@@
 			)
 		)
-		(property "MPN" "0402WGF330JTCE"
+		(property "MPN" "RC-01W33R0FT"
 			(at 119.38 177.8 0)
 			(hide yes)
@@
 			)
 		)
-		(property "LCSC" "C25105"
+		(property "LCSC" "C320843"
 			(at 119.38 88.9 0)
 			(hide yes)
@@
 			)
 		)
-		(property "MPN" "0402WGF330JTCE"
+		(property "MPN" "RC-01W33R0FT"
 			(at 119.38 88.9 0)
 			(hide yes)
@@
 			)
 		)
-		(property "LCSC" "C25105"
+		(property "LCSC" "C320843"
 			(at 129.54 177.8 0)
 			(hide yes)
@@
 			)
 		)
-		(property "MPN" "0402WGF330JTCE"
+		(property "MPN" "RC-01W33R0FT"
 			(at 129.54 177.8 0)
 			(hide yes)

Commit message: Design-review fixes: core buck feed-forward, EPWM2A/B pull-downs, mux bypass
From the pre-order design review:
- C77 120 pF C0G (C40059) across R1, VCC_SENSE_P to FB_0V75: the AP61302
  datasheet requires a feed-forward cap (33 pF with a 200k top resistor;
  scaled for R1 = 49.9k).
- C4, C7 22 pF -> 33 pF (C1562), the AP61102 datasheet value for these
  dividers.
- R40, R41 10k 0201 pull-downs on EPWM2A / EPWM2B. These drive the power
  board's Si8661 isolator inputs, which have no pull-down there; the other
  PWM lines already have 10k pull-downs on the power board.
- C78, C79 100 nF extra +3V3A bypass for the muxes (C79 is placed near U14;
  move it to U13 pin 16 if it's meant for U13).
Parts placed by hand; new reference text hidden like the rest.

DRC: 0 errors, 0 unconnected, 0 parity issues. BOM 44 lines / 146 parts;
all parts orderable for 10 boards (tightest ADS7056, 29).

Co-Authored-By: Claude Opus 5.5 <noreply@anthropic.com>
Parts:
- added C78, C79: 100n, Capacitor_SMD:C_0402_1005Metric, symbol Device:C
Connections:
- net +3V3A: now also C78.1, C79.1
- net GND: now also C78.2, C79.2

Commit message: BOM: secure 680p stock, two extended parts to basic
- C56, C61 (680 pF C0G kickback): 0402CG681J500NT (C301953, 78 orderable)
  -> Yageo CC0402JRNPO9BN681 (C113781, 57063 orderable), same spec.
- C77 core feed-forward 120 pF (C40059, extended) -> 100 pF C0G basic
  (C1546); zero moves from 24 to 31 kHz.
- R1 core divider top 49.9k (C137969, extended) -> 51k basic (C25794);
  core output 0.750 -> 0.753 V (+0.4 %, FPGA allows +/-3 %).
Extended part types 25 -> 23. Schematic and board updated together;
docs updated for 51k/0.753 V. Five symbols added earlier re-indented.

DRC: 0 errors, 0 unconnected, 0 parity issues. ERC: GNDSENSE only.

Co-Authored-By: Claude Opus 5.5 <noreply@anthropic.com>
Parts:
- C56, C61: LCSC C301953 -> C113781; MPN 0402CG681J500NT -> CC0402JRNPO9BN681
Changed lines of the file:
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@@
 			)
 		)
-		(property "LCSC" "C301953"
+		(property "LCSC" "C113781"
 			(at 162.56 127 0)
 			(hide yes)
@@
 			)
 		)
-		(property "MPN" "0402CG681J500NT"
+		(property "MPN" "CC0402JRNPO9BN681"
 			(at 162.56 127 0)
 			(hide yes)
@@
 			)
 		)
-		(property "LCSC" "C301953"
+		(property "LCSC" "C113781"
 			(at 162.56 38.1 0)
 			(hide yes)
@@
 			)
 		)
-		(property "MPN" "0402CG681J500NT"
+		(property "MPN" "CC0402JRNPO9BN681"
 			(at 162.56 38.1 0)
 			(hide yes)
@@
 		)
 	)
-		(symbol
+	(symbol
 		(lib_id "Device:C")
 		(at 63.5 215.9 0)
@@
 		)
 	)
-		(symbol
+	(symbol
 		(lib_id "Device:C")
 		(at 76.2 215.9 0)
