File: hardware/sheets/connector.kicad_sch (KiCad schematic)
At the start: 9 parts, among them J1 Power board

Commit message: Design-review fixes: core buck feed-forward, EPWM2A/B pull-downs, mux bypass
From the pre-order design review:
- C77 120 pF C0G (C40059) across R1, VCC_SENSE_P to FB_0V75: the AP61302
  datasheet requires a feed-forward cap (33 pF with a 200k top resistor;
  scaled for R1 = 49.9k).
- C4, C7 22 pF -> 33 pF (C1562), the AP61102 datasheet value for these
  dividers.
- R40, R41 10k 0201 pull-downs on EPWM2A / EPWM2B. These drive the power
  board's Si8661 isolator inputs, which have no pull-down there; the other
  PWM lines already have 10k pull-downs on the power board.
- C78, C79 100 nF extra +3V3A bypass for the muxes (C79 is placed near U14;
  move it to U13 pin 16 if it's meant for U13).
Parts placed by hand; new reference text hidden like the rest.

DRC: 0 errors, 0 unconnected, 0 parity issues. BOM 44 lines / 146 parts;
all parts orderable for 10 boards (tightest ADS7056, 29).

Co-Authored-By: Claude Opus 5.5 <noreply@anthropic.com>
Parts:
- added R40, R41: 10k, Resistor_SMD:R_0201_0603Metric, symbol Device:R
Connections:
- net EPWM2A: now also R40.1
- net EPWM2B: now also R41.1
- net GND: now also R40.2, R41.2
