File: hardware/sheets/power.kicad_sch (KiCad schematic)
At the start: 37 parts, among them U16 TLV75518PDBVR, U2 AP61302Z6-7, U3 AP61102Z6-7, U4 AP61102Z6-7, U5 TLV75512PDBVR, U6 TLV75533PDBVR

Commit message: R1 (core buck feedback 49.9k): Yageo RC0402FR-0749K9L
The UniOhm 0402WGF4992TCE (C25897) showed 831 in stock but -38942 orderable
at JLC (oversold) with a 9023-piece minimum. Replaced by RC0402FR-0749K9L
(C137969, 0402 49.9k 1 %, 1.28M orderable, no minimum) in the schematic and
on the board. Core voltage unchanged.

Every part in the final BOM now has orderable stock for 10 boards and a
minimum purchase of 1; tightest is ADS7056 (34 orderable, 2 per board).

Co-Authored-By: Claude Opus 5.5 <noreply@anthropic.com>
Parts:
- R1: LCSC C25897 -> C137969; MPN 0402WGF4992TCE -> RC0402FR-0749K9L
Changed lines of the file:
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@@
 			)
 		)
-		(property "LCSC" "C25897"
+		(property "LCSC" "C137969"
 			(at 93.98 38.1 0)
 			(hide yes)
@@
 			)
 		)
-		(property "MPN" "0402WGF4992TCE"
+		(property "MPN" "RC0402FR-0749K9L"
 			(at 93.98 38.1 0)
 			(hide yes)

Commit message: Design-review fixes: core buck feed-forward, EPWM2A/B pull-downs, mux bypass
From the pre-order design review:
- C77 120 pF C0G (C40059) across R1, VCC_SENSE_P to FB_0V75: the AP61302
  datasheet requires a feed-forward cap (33 pF with a 200k top resistor;
  scaled for R1 = 49.9k).
- C4, C7 22 pF -> 33 pF (C1562), the AP61102 datasheet value for these
  dividers.
- R40, R41 10k 0201 pull-downs on EPWM2A / EPWM2B. These drive the power
  board's Si8661 isolator inputs, which have no pull-down there; the other
  PWM lines already have 10k pull-downs on the power board.
- C78, C79 100 nF extra +3V3A bypass for the muxes (C79 is placed near U14;
  move it to U13 pin 16 if it's meant for U13).
Parts placed by hand; new reference text hidden like the rest.

DRC: 0 errors, 0 unconnected, 0 parity issues. BOM 44 lines / 146 parts;
all parts orderable for 10 boards (tightest ADS7056, 29).

Co-Authored-By: Claude Opus 5.5 <noreply@anthropic.com>
Parts:
- added C77: 120p, Capacitor_SMD:C_0402_1005Metric, symbol Device:C
- C4, C7: value 22p -> 33p; LCSC C1555 -> C1562; MPN 0402CG220J500NT -> 0402CG330J500NT
Connections:
- net FB_0V75: now also C77.2
- net VCC_SENSE_P: now also C77.1
Changed lines of the file:
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@@
 			)
 		)
-		(property "Value" "22p"
+		(property "Value" "33p"
 			(at 124.46 74.93 0)
 			(show_name no)
@@
 			)
 		)
-		(property "LCSC" "C1555"
+		(property "LCSC" "C1562"
 			(at 121.92 73.66 0)
 			(hide yes)
@@
 			)
 		)
-		(property "MPN" "0402CG220J500NT"
+		(property "MPN" "0402CG330J500NT"
 			(at 121.92 73.66 0)
 			(hide yes)
@@
 			)
 		)
-		(property "Value" "22p"
+		(property "Value" "33p"
 			(at 124.46 110.49 0)
 			(show_name no)
@@
 			)
 		)
-		(property "LCSC" "C1555"
+		(property "LCSC" "C1562"
 			(at 121.92 109.22 0)
 			(hide yes)
@@
 			)
 		)
-		(property "MPN" "0402CG220J500NT"
+		(property "MPN" "0402CG330J500NT"
 			(at 121.92 109.22 0)
 			(hide yes)
@@
 		)
 	)
+		(symbol
+		(lib_id "Device:C")
+		(at 63.5 215.9 0)
+		(unit 1)
+		(body_style 1)
+		(exclude_from_sim no)
+		(in_bom yes)
+		(on_board yes)
+		(in_pos_files yes)
+		(dnp no)
+		(property "Reference" "C77"
+			(at 66.04 214.63 0)
+			(show_name no)
+			(do_not_autoplace no)
+			(effects
+				(font
+					(size 1.27 1.27)
+				)
+				(justify left)
+			)
+		)
+		(property "Value" "120p"
+			(at 66.04 217.17 0)
+			(show_name no)
+			(do_not_autoplace no)
+			(effects
+				(font
+					(size 1.27 1.27)
+				)
+				(justify left)
+			)
+		)
+		(property "Footprint" "Capacitor_SMD:C_0402_1005Metric"
+			(at 63.5 215.9 0)
+			(hide yes)
+			(show_name no)
+			(do_not_autoplace no)
+			(effects
+				(font
+					(size 1.27 1.27)
+				)
+				(justify left)
+			)
+		)
+		(property "Datasheet" ""
+			(at 63.5 215.9 0)
+			(hide yes)
+			(show_name no)
+			(do_not_autoplace no)
+			(effects
+				(font
+					(size 1.27 1.27)
+				)
+				(justify left)
+			)
+		)
+		(property "Description" "Feed-forward"
+			(at 63.5 215.9 0)
+			(hide yes)
+			(show_name no)
+			(do_not_autoplace no)
+			(effects
+				(font
+					(size 1.27 1.27)
+				)
+				(justify left)
+			)
+		)
+		(property "LCSC" "C40059"
+			(at 63.5 215.9 0)
+			(hide yes)
+			(show_name no)
+			(do_not_autoplace no)
+			(effects
+				(font
+					(size 1.27 1.27)
+				)
+				(justify left)
+			)
+		)
+		(property "MPN" "0402CG121J500NT"
+			(at 63.5 215.9 0)
+			(hide yes)
+			(show_name no)
+			(do_not_autoplace no)
+			(effects
+				(font
+					(size 1.27 1.27)
+				)
+				(justify left)
+			)
+		)
+		(pin "1"
+		)
+		(pin "2"
+		)
+		(instances
+			(project "control_card"
+				(path "/02cf0cd1-c66b-5c4c-858e-ca84c1bbaba4/affdd0cf-ed48-5605-8b8d-7bdc9d18f6df"
+					(reference "C77")
+					(unit 1)
+				)
+			)
+		)
+	)
+	(global_label "VCC_SENSE_P"
+		(shape passive)
+		(at 63.5 212.09 90)
+		(fields_autoplaced yes)
+		(effects
+			(font
+				(size 1.27 1.27)
+			)
+			(justify left)
+		)
+		(property "Intersheetrefs" "${INTERSHEET_REFS}"
+			(at 63.5 212.09 0)
+			(hide yes)
+			(show_name no)
+			(do_not_autoplace no)
+			(effects
+				(font
+					(size 1.27 1.27)
+				)
+			)
+		)
+	)
+	(label "FB_0V75"
+		(at 63.5 219.71 270)
+		(effects
+			(font
+				(size 1.27 1.27)
+			)
+			(justify right bottom)
+		)
+	)

Commit message: BOM: secure 680p stock, two extended parts to basic
- C56, C61 (680 pF C0G kickback): 0402CG681J500NT (C301953, 78 orderable)
  -> Yageo CC0402JRNPO9BN681 (C113781, 57063 orderable), same spec.
- C77 core feed-forward 120 pF (C40059, extended) -> 100 pF C0G basic
  (C1546); zero moves from 24 to 31 kHz.
- R1 core divider top 49.9k (C137969, extended) -> 51k basic (C25794);
  core output 0.750 -> 0.753 V (+0.4 %, FPGA allows +/-3 %).
Extended part types 25 -> 23. Schematic and board updated together;
docs updated for 51k/0.753 V. Five symbols added earlier re-indented.

DRC: 0 errors, 0 unconnected, 0 parity issues. ERC: GNDSENSE only.

Co-Authored-By: Claude Opus 5.5 <noreply@anthropic.com>
Parts:
- C77: value 120p -> 100p; LCSC C40059 -> C1546; MPN 0402CG121J500NT -> 0402CG101J500NT
- R1: value 49k9 -> 51k; LCSC C137969 -> C25794; MPN RC0402FR-0749K9L -> 0402WGF5102TCE
Changed lines of the file:
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@@
 			)
 		)
-		(property "Value" "49k9"
+		(property "Value" "51k"
 			(at 96.52 39.37 0)
 			(show_name no)
@@
 			)
 		)
-		(property "LCSC" "C137969"
+		(property "LCSC" "C25794"
 			(at 93.98 38.1 0)
 			(hide yes)
@@
 			)
 		)
-		(property "MPN" "RC0402FR-0749K9L"
+		(property "MPN" "0402WGF5102TCE"
 			(at 93.98 38.1 0)
 			(hide yes)
@@
 		)
 	)
-		(symbol
+	(symbol
 		(lib_id "Device:C")
 		(at 63.5 215.9 0)
@@
 			)
 		)
-		(property "Value" "120p"
+		(property "Value" "100p"
 			(at 66.04 217.17 0)
 			(show_name no)
@@
 			)
 		)
-		(property "LCSC" "C40059"
+		(property "LCSC" "C1546"
 			(at 63.5 215.9 0)
 			(hide yes)
@@
 			)
 		)
-		(property "MPN" "0402CG121J500NT"
+		(property "MPN" "0402CG101J500NT"
 			(at 63.5 215.9 0)
 			(hide yes)
