File: hardware/sheets/power.kicad_sch (KiCad schematic)
At the start: 38 parts, among them U16 TLV75518PDBVR, U2 AP61302Z6-7, U3 AP61102Z6-7, U4 AP61102Z6-7, U5 TLV75512PDBVR, U6 TLV75533PDBVR

Commit message: remove ldos and replace with switchers
Parts:
- removed C10, C74: 1u, Capacitor_SMD:C_0402_1005Metric, symbol Device:C
- removed U16: TLV75518PDBVR, Package_TO_SOT_SMD:SOT-23-5, symbol Regulator_Linear:TLV75518PDBV
- removed U5: TLV75512PDBVR, Package_TO_SOT_SMD:SOT-23-5, symbol Regulator_Linear:TLV75512PDBV
- added C80, C83: 33p, Capacitor_SMD:C_0402_1005Metric, symbol Device:C
- added C81, C84: 10u, Capacitor_SMD:C_0603_1608Metric, symbol Device:C
- added C82, C85: 22u, Capacitor_SMD:C_0603_1608Metric, symbol Device:C
- added L4, L5: 1u, Inductor_SMD:L_Cenker_CKCS201610, symbol Device:L
- added R42, R43, R44, R47, R48, R49, R51: 200k, Resistor_SMD:R_0402_1005Metric, symbol Device:R
- added R45, R46, R50: 100k, Resistor_SMD:R_0402_1005Metric, symbol Device:R
- added U17, U18: AP61102Z6-7, Package_TO_SOT_SMD:SOT-563, symbol Regulator_Switching:AP61202Z6
Connections:
- net +1V2: now also C80.1, C82.1, L4.2, R42.1
- net +1V8_HR: now also C83.1, C85.1, L5.2, R44.1
- net +5V: now also C81.1, C84.1, R46.1, R50.1, U17.3 (VIN), U18.3 (VIN); no longer U2.5 (EN)
- net GND: now also C81.2, C82.2, C84.2, C85.2, R43.2, R45.2, R47.2, R48.2, R49.2, R51.2, U17.2 (GND), U18.2 (GND)
- net PG_0V75: now also R48.1
- net PG_1V8: now also R49.1
- net PG_3V3: now reaches U4.6 (PG)
- net PG_3V3: now also R50.2, R51.1, U17.5 (EN), U18.5 (EN)
- new net EN_0V75: R46.2, R47.1, U2.5 (EN)
- new net FB_1V2: C80.2, R42.2, R43.1, U17.1 (FB)
- new net FB_1V8HR: C83.2, R44.2, R45.1, U18.1 (FB)
- new net SW_1V2: L4.1, U17.4 (SW)
- new net SW_1V8HR: L5.1, U18.4 (SW)
- no-connect marks 4 -> 3
Other:
- note added: "Power-up order: 0.75 V -> PG -> 1.8 V -> PG -> 3.3 V -> PG -> 1.2 V and 1.8 V (HR). Forced PWM: EN below VIN - 200 mV (100k up / 200k down = 3.33 V); EN at VIN would select PFM at light load. Buck FB reference 0.6 V: Vout = 0.6 x (1 + Rtop/Rbot). AP61102/AP61302 pinout: FB, GND, VIN, SW, EN, PG. Core divider top sits on VCC_SENSE_P (FPGA VCCLSENSE ball, remote sense); 100R from +0V75 keeps regula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"
- note removed: "Power-up order (proven on agilex3_control_card_v1): 0.75 V -> PG -> 1.8 V -> PG -> 3.3 V and 1.2 V. Buck FB reference 0.6 V: Vout = 0.6 x (1 + Rtop/Rbot). AP61102/AP61302 pinout: FB, GND, VIN, SW, EN, PG. Core divider top sits on VCC_SENSE_P (FPGA VCCLSENSE ball, remote sense); 100R from +0V75 keeps regulation if open."
- title: Power: 5 V in, 0.75/1.8/3.3 V bucks, 1.2 V and analog 3.3 V LDOs -> Power: 5 V in, 0.75/1.8/3.3/1.2/1.8 V (HR) bucks, analog 3.3 V LDO

Commit message: finish placing components
Parts:
- removed C14: 22u, Capacitor_SMD:C_0805_2012Metric, symbol Device:C
- R46: footprint Resistor_SMD:R_0402_1005Metric -> Resistor_SMD:R_0201_0603Metric
Changed lines of the file:
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@@
 	(wire
 		(pts
-			(xy 27.94 184.15) (xy 27.94 186.69)
-		)
-		(stroke
-			(width 0)
-			(type default)
-		)
-	)
-	(wire
-		(pts
 			(xy 55.88 45.72) (xy 58.42 45.72)
 		)
@@
 	(wire
 		(pts
-			(xy 27.94 176.53) (xy 27.94 173.99)
-		)
-		(stroke
-			(width 0)
-			(type default)
-		)
-	)
-	(wire
-		(pts
 			(xy 347.98 77.47) (xy 347.98 80.01)
 		)
@@
 		)
 	)
-	(global_label "+5V"
-		(shape passive)
-		(at 27.94 173.99 90)
-		(fields_autoplaced yes)
-		(effects
-			(font
-				(size 1.27 1.27)
-			)
-			(justify left)
-		)
-		(property "Intersheetrefs" "${INTERSHEET_REFS}"
-			(at 27.94 173.99 0)
-			(hide yes)
-			(show_name no)
-			(do_not_autoplace no)
-			(effects
-				(font
-					(size 1.27 1.27)
-				)
-			)
-		)
-	)
 	(global_label "+1V8_ADC"
 		(shape passive)
@@
 		)
 	)
-	(global_label "GND"
-		(shape passive)
-		(at 27.94 186.69 270)
-		(fields_autoplaced yes)
-		(effects
-			(font
-				(size 1.27 1.27)
-			)
-			(justify right)
-		)
-		(property "Intersheetrefs" "${INTERSHEET_REFS}"
-			(at 27.94 186.69 0)
-			(hide yes)
-			(show_name no)
-			(do_not_autoplace no)
-			(effects
-				(font
-					(size 1.27 1.27)
-				)
-			)
-		)
-	)
 	(global_label "+5V"
 		(shape passive)
@@
 			)
 		)
-		(property "Footprint" "Resistor_SMD:R_0402_1005Metric"
+		(property "Footprint" "Resistor_SMD:R_0201_0603Metric"
 			(at 254 152.4 0)
 			(hide yes)
@@
 					(unit 1)
 				)
-			)
-		)
-	)
-	(symbol
-		(lib_id "Device:C")
-		(at 27.94 180.34 0)
-		(unit 1)
-		(body_style 1)
-		(exclude_from_sim no)
-		(in_bom yes)
-		(on_board yes)
-		(in_pos_files yes)
-		(dnp no)
-		(property "Reference" "C14"
-			(at 30.48 179.07 0)
-			(show_name no)
-			(do_not_autoplace no)
-			(effects
-				(font
-					(size 1.27 1.27)
-				)
-				(justify left)
-			)
-		)
-		(property "Value" "22u"
-			(at 30.48 181.61 0)
-			(show_name no)
-			(do_not_autoplace no)
-			(effects
-				(font
-					(size 1.27 1.27)
-				)
-				(justify left)
-			)
-		)
-		(property "Footprint" "Capacitor_SMD:C_0805_2012Metric"
-			(at 27.94 180.34 0)
-			(hide yes)
-			(show_name no)
-			(do_not_autoplace no)
-			(effects
-				(font
-					(size 1.27 1.27)
-				)
-				(justify left)
-			)
-		)
-		(property "Datasheet" ""
-			(at 27.94 180.34 0)
-			(hide yes)
-			(show_name no)
-			(do_not_autoplace no)
-			(effects
-				(font
-					(size 1.27 1.27)
-				)
-				(justify left)
-			)
-		)
-		(property "Description" "5 V input from J1"
-			(at 27.94 180.34 0)
-			(hide yes)
-			(show_name no)
-			(do_not_autoplace no)
-			(effects
-				(font
-					(size 1.27 1.27)
-				)
-				(justify left)
-			)
-		)
-		(property "LCSC" "C45783"
-			(at 27.94 180.34 0)
-			(hide yes)
-			(show_name no)
-			(do_not_autoplace no)
-			(effects
-				(font
-					(size 1.27 1.27)
-				)
-				(justify left)
-			)
-		)
-		(property "MPN" "CL21A226MAQNNNE"
-			(at 27.94 180.34 0)
-			(hide yes)
-			(show_name no)
-			(do_not_autoplace no)
-			(effects
-				(font
-					(size 1.27 1.27)
-				)
-				(justify left)
-			)
-		)
-		(property "Group" "input_5v"
-			(at 27.94 180.34 0)
-			(hide yes)
-			(show_name no)
-			(do_not_autoplace no)
-			(effects
-				(font
-					(size 1.27 1.27)
-				)
-				(justify left)
-			)
-		)
-		(pin "1"
-		)
-		(pin "2"
-		)
-		(instances
-			(project "control_card"
-				(path "/02cf0cd1-c66b-5c4c-858e-ca84c1bbaba4/affdd0cf-ed48-5605-8b8d-7bdc9d18f6df"
-					(reference "C14")
-					(unit 1)
-				)
