File: hardware/sheets/power.kicad_sch (KiCad schematic)
At the start: 53 parts, among them U17 AP61102Z6-7, U18 AP61102Z6-7, U2 AP61302Z6-7, U3 AP61102Z6-7, U4 AP61102Z6-7, U6 TLV75533PDBVR

Commit message: Switcher pours, GND to U2/U17/U18 pins, R46 0201 part
B.Cu zones for the SW, output, GND and +5V nodes of all four AP61x02 cells,
with distinct priorities (equal-priority overlaps hang the KiCad 10 filler).
Ground pours extended to the switcher GND pins. Removed a dangling GND stub,
a PG_0V75 via in U2's pad and a dangling +1V2 via; reference designators
hidden again. R46 sits on an 0201 footprint: part changed to 0201WMF1003TEE
(C270364). DRC: 0 errors, 0 unconnected, 0 parity issues.

Co-Authored-By: Claude Opus 5.5 <noreply@anthropic.com>
Parts:
- R46: LCSC C25741 -> C270364; MPN 0402WGF1003TCE -> 0201WMF1003TEE
Changed lines of the file:
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@@
 			)
 		)
-		(property "LCSC" "C25741"
+		(property "LCSC" "C270364"
 			(at 254 152.4 0)
 			(hide yes)
@@
 			)
 		)
-		(property "MPN" "0402WGF1003TCE"
+		(property "MPN" "0201WMF1003TEE"
 			(at 254 152.4 0)
 			(hide yes)

Commit message: R46: RC0201FR-07100KL (C106224)
0201WMF1003TEE (C270364) went oversold: -58871 orderable, minimum
purchase 10026. Same value, size and tolerance.

Co-Authored-By: Claude Opus 5.5 <noreply@anthropic.com>
Parts:
- R46: LCSC C270364 -> C106224; MPN 0201WMF1003TEE -> RC0201FR-07100KL
Changed lines of the file:
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@@
 			)
 		)
-		(property "LCSC" "C270364"
+		(property "LCSC" "C106224"
 			(at 254 152.4 0)
 			(hide yes)
@@
 			)
 		)
-		(property "MPN" "0201WMF1003TEE"
+		(property "MPN" "RC0201FR-07100KL"
 			(at 254 152.4 0)
 			(hide yes)
