File: hardware/sheets/fpga_io.kicad_sch (KiCad schematic)
At the start: 1 part, among them U1 A3CZ065BB18AE7S

Commit message: remove ldos and replace with switchers
Connections:
- net J1_P28: now also U1.BN16 (6F_IO_HVIO_6F_1_TXCLK1_Data_Ctrl1); no longer U1.BN19 (6A_IO_HVIO_6A_19_TXCLK19_Data_Ctrl19)
Changed lines of the file:
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@@
-	)
-	(no_connect
-		(at 652.78 40.64)
 	)
 	(no_connect
@@
 	)
 	(no_connect
+		(at 129.54 86.36)
+	)
+	(no_connect
 		(at 342.9 86.36)
 	)
@@
 	(wire
 		(pts
-			(xy 129.54 86.36) (xy 127 86.36)
-		)
-		(stroke
-			(width 0)
-			(type default)
-		)
-	)
-	(wire
-		(pts
 			(xy 147.32 215.9) (xy 149.86 215.9)
 		)
@@
 		)
 	)
+	(global_label "J1_P28"
+		(shape passive)
+		(at 652.78 40.64 180)
+		(fields_autoplaced yes)
+		(effects
+			(font
+				(size 1.27 1.27)
+			)
+			(justify right)
+		)
+		(property "Intersheetrefs" "${INTERSHEET_REFS}"
+			(at 652.78 40.64 0)
+			(hide yes)
+			(show_name no)
+			(do_not_autoplace no)
+			(effects
+				(font
+					(size 1.27 1.27)
+				)
+			)
+		)
+	)
 	(global_label "ADBSEL1"
 		(shape passive)
@@
 			(hide yes)
 			(show_name no)
-			(do_not_autoplace no)
-			(effects
-				(font
-					(size 1.27 1.27)
-				)
-			)
-		)
-	)
-	(global_label "J1_P28"
-		(shape passive)
-		(at 127 86.36 180)
-		(fields_autoplaced yes)
-		(effects
-			(font
-				(size 1.27 1.27)
-			)
-			(justify right)
-		)
-		(property "Intersheetrefs" "${INTERSHEET_REFS}"
-			(at 127 86.36 0)
-			(hide yes)
-			(show_name no)
